File: hardware/e7_cart/vmw-e7/vmw-e7.kicad_pcb (KiCad board)
At the start: 2 copper layers, 70.6 x 95.2 mm, 8 parts, among them J1 Conn_01x02_Pin, J2 Conn_01x02_Pin, U1 E7, U2 ROM, U3 ROM, U4 SRAM, U5 2600Cartridge

Commit message: e7: update
Parts:
- moved J2 10.0 mm to (122.0, 108.8), turned to 180 degrees
- moved C1 8.80 mm to (134.0, 108.5)
- moved J1 5.87 mm to (97.5, 84.0)
- moved U4 3.44 mm to (133.5, 83.4)
- moved U2 2.15 mm to (133.7, 76.5)
- moved U1 1.81 mm to (155.7, 96.6)
- moved U3 0.49 mm to (111.9, 76.4)
Routing:
- net D4: track 0.00 -> 23.1 mm
- net A7R: track 0.00 -> 23.1 mm
- net D3: track 0.00 -> 23.1 mm
- net A12ROM_A9RAM: track 0.00 -> 23.0 mm
- net A8: track 0.00 -> 23.0 mm
- net A5R: track 0.00 -> 23.0 mm
- net A4R: track 0.00 -> 23.0 mm
- net A3R: track 0.00 -> 22.9 mm
- net A2R: track 0.00 -> 22.9 mm
- net A1R: track 0.00 -> 22.9 mm
- net A0R: track 0.00 -> 22.8 mm
- net D0: track 0.00 -> 22.8 mm
- net A6R: track 0.00 -> 22.8 mm
- net D7: track 0.00 -> 22.8 mm
- net D2: track 0.00 -> 22.8 mm
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
Commit message: e7: more work on pcb
Parts:
- moved C1 39.2 mm to (98.0, 92.9)
- moved J2 31.1 mm to (94.6, 94.1)
- moved J1 13.5 mm to (99.1, 97.4)
- moved U1 3.56 mm to (158.4, 94.2)
- moved U4 2.89 mm to (135.9, 85.0)
- moved U2 2.78 mm to (136.5, 76.5)
Routing:
- net GNDREF: track 0.00 -> 268.3 mm, vias 0 -> 1
- net D3: track 23.1 -> 180.4 mm
- net D4: track 23.1 -> 170.7 mm
- net D5: track 22.8 -> 161.0 mm
- net VCC: track 0.00 -> 122.4 mm, vias 0 -> 1
- net A7: track 0.00 -> 79.4 mm, vias 0 -> 1
- net A6: track 0.00 -> 75.6 mm, vias 0 -> 1
- net A5: track 0.00 -> 72.0 mm, vias 0 -> 1
- net A4: track 0.00 -> 69.3 mm, vias 0 -> 1
- net A3: track 0.00 -> 66.7 mm, vias 0 -> 1
- net A2: track 0.00 -> 64.5 mm, vias 0 -> 1
- net A1: track 0.00 -> 62.0 mm, vias 0 -> 1
- net D7: track 22.8 -> 83.5 mm
- net A0: track 0.00 -> 58.0 mm, vias 0 -> 1
- net D6: track 22.8 -> 77.3 mm
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Other:
- rule pad_to_mask_clearance: 0 -> 0.0508

Commit message: e7: pbc mostly done
Parts:
- moved J1 37.3 mm to (135.6, 104.5), turned to -90 degrees
- moved J2 17.1 mm to (108.2, 104.6), turned to 90 degrees
Routing:
- net A9: track 25.5 -> 135.7 mm, vias 0 -> 1
- net A8: track 35.0 -> 133.6 mm, vias 0 -> 2
- net A10: track 49.9 -> 146.2 mm, vias 0 -> 6
- net A11: track 0.00 -> 88.3 mm, vias 0 -> 1
- net A10RAM: track 22.7 -> 97.2 mm, vias 0 -> 3
- net D2: track 70.9 -> 141.4 mm
- net A11ROM_A8RAM: track 25.5 -> 95.1 mm, vias 0 -> 2
- net D1: track 70.8 -> 138.4 mm
- net D0: track 70.8 -> 136.0 mm
- net A1R: track 32.5 -> 97.4 mm, vias 0 -> 2
- net A12ROM_A9RAM: track 25.8 -> 85.1 mm, vias 0 -> 2
- net A3R: track 32.5 -> 91.3 mm, vias 0 -> 1
- net A2R: track 32.7 -> 84.6 mm, vias 0 -> 3
- net D6: track 77.3 -> 129.1 mm, vias 0 -> 1
- net D7: track 83.5 -> 134.1 mm, vias 0 -> 1
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